File: kicad/fc-brushed-aio-rev-a/fc-brushed-aio-rev-a.kicad_pcb (KiCad board)
At the start: 4 copper layers, 34.7 x 34.7 mm, 115 parts, among them J1 Battery, J10 USART1, J11 USART2, J12 FC-ESC con, J13 Motors2, J14 UART4, J15 USART6, J2 M1, J3 M2, J4 M3, J5 M4, J6 M5, J7 M6, J8 M7, J9 M8, Q1 PMOS, Q2 2300A, Q3 2300A, Q4 2300A, Q5 2300A, Q6 2300A, Q7 2300A, Q8 2300A, Q9 2300A, SW1 SW_SPST, U1 STM32F405RGTx, U13 W25Q128JVS, U14 INA180A3, U2 BMP388, U3 BMI270, U4 TPS62172DSG, U5 GT-USB-7010AN, Y1 8 MHz

Commit message: More progress on pcb!
Parts:
- removed kibuzzard-66DDC02B: G***, kibuzzard-66DDC02B
- removed kibuzzard-66DDC032: G***, kibuzzard-66DDC032
- removed kibuzzard-66DDC060 (x2): G***, kibuzzard-66DDC060
- removed kibuzzard-66DDC064 (x2): G***, kibuzzard-66DDC064
- removed kibuzzard-66DDC0AE: G***, kibuzzard-66DDC0AE
- removed kibuzzard-66DDC0BA: G***, kibuzzard-66DDC0BA
- removed kibuzzard-66DDC0C2: G***, kibuzzard-66DDC0C2
- removed kibuzzard-66DDC0DD: G***, kibuzzard-66DDC0DD
- removed kibuzzard-66DDC0E1: G***, kibuzzard-66DDC0E1
- removed kibuzzard-66DDC0E5: G***, kibuzzard-66DDC0E5
- added J16: I2C, custom:Conn_4_Accesory, F.Cu at (173.1, 114.9)
- added J17: I2C, custom:Conn_4_Accesory, F.Cu at (175.1, 110.3)
- added J18: I2C, custom:Conn_4_Accesory, F.Cu at (169.8, 110.3)
- added J19: Debug, Connector_PinHeader_1.27mm:PinHeader_1x03_P1.27mm_Vertical, B.Cu at (182.8, 120.9)
- added kibuzzard-66E3374B: G***, kibuzzard-66E3374B, F.Cu at (161.3, 110.4)
- moved J11 31.9 mm to (164.0, 137.8), turned to -90 degrees
- moved J14 30.3 mm to (169.8, 108.0)
- moved J10 15.2 mm to (175.1, 108.0)
- moved J12 6.60 mm to (158.6, 108.0)
- moved J13 5.00 mm to (165.4, 110.3), turned to -90 degrees
- moved D4 1.35 mm to (174.1, 123.1)
- moved J15 0.54 mm to (159.2, 137.8), turned to -90 degrees
- moved C6 0.51 mm to (165.9, 114.3)
- moved R13 0.40 mm to (165.6, 115.8)
- moved R2 0.40 mm to (175.8, 118.9)
- moved R3 0.40 mm to (174.9, 118.9)
- moved C24 0.30 mm to (154.9, 114.7)
- moved D5 0.25 mm to (179.8, 131.9)
- moved D9 0.25 mm to (179.8, 129.6)
- moved C20 0.20 mm to (154.9, 113.9)
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Connections:
- J11 pad 1: TX2 -> TX6
- J11 pad 2: RX2 -> RX6
- J12 pad 3: Current -> CURR_EXT
- J15 pad 1: TX6 -> TX2
- J15 pad 2: RX6 -> RX2
- U1 pad 35: unconnected-(U1-PB14-Pad35) -> RGB_LED
- U1 pad 41: unconnected-(U1-PA8-Pad41) -> SERVO_1
- U1 pad 50: unconnected-(U1-PA15-Pad50) -> SERVO_2
- U1 pad 55: unconnected-(U1-PB3-Pad55) -> SERVO_3
- U1 pad 8: unconnected-(U1-PC0-Pad8) -> CURR_EXT
Routing:
- net +3V3: track 5.04 -> 96.0 mm, vias 0 -> 12
- net VBAT+: track 8.44 -> 45.8 mm, vias 1 -> 2
- net M2: track 12.9 -> 46.9 mm, vias 2 -> 3
- net M3: track 12.6 -> 45.6 mm, vias 2 -> 4
- net M1: track 14.7 -> 46.3 mm, vias 2 -> 4
- net M7: track 10.3 -> 39.7 mm, vias 2 -> 5
- net M6: track 10.8 -> 36.8 mm, vias 2 -> 4
- net RGB_LED: track 0.00 -> 21.7 mm, vias 0 -> 2
- net M5: track 9.11 -> 30.5 mm, vias 2 -> 4
- net SERVO_2: track 0.00 -> 19.5 mm, vias 0 -> 2
- net VBUS: track 35.6 -> 17.5 mm
- net TX6: track 0.00 -> 18.0 mm, vias 0 -> 2
- net RX6: track 0.00 -> 17.8 mm, vias 0 -> 2
- net SERVO_1: track 0.00 -> 16.5 mm, vias 0 -> 2
- net CURR_SENSE: track 2.44 -> 17.2 mm, vias 2 -> 3
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Other:
- board text added: "1"
- board text added: "2"
- board text added: "3"
- board text added: "3V"
- board text added: "4"
- board text added: "5"
- board text added: "6"
- board text added: "7"
- board text added: "8"
- board text added: "C"
- board text added: "CL"
- board text added: "DA"
- board text added: "G"
- board text added: "L"
- board text added: "R1"
- board text added: "R2"
- board text added: "R4"
- board text added: "R6"
- board text added: "S1"
- board text added: "S2"
- board text added: "S3"
- board text added: "T"
- board text added: "T1"
- board text added: "T2"
- board text added: "T4"
- board text added: "T6"
- board text added: "V"
- board text removed: "M1"

Commit message: Majority of routing complete. Schematic too.
Parts:
- added C25: 2.2uF, custom:C_0402_1005Metric_NoSilk, F.Cu at (169.5, 130.2)
- added C26: 2.2uF, custom:C_0402_1005Metric_NoSilk, F.Cu at (173.8, 118.9)
- R4, R5, R6: value 330R -> 1k
- moved C16 0.25 mm to (159.2, 125.2)
- moved R7 0.20 mm to (158.3, 126.9)
- moved R8 0.20 mm to (159.2, 126.9)
- moved C9 0.05 mm to (172.5, 118.5)
Connections:
- J12 pad 1: VBAT+ -> VBAT
- J19 pad 1: SWDIO -> SWCLK
- J19 pad 2: SWCLK -> SWDIO
- U1 pad 31: unconnected-(U1-VCAP_1-Pad31) -> Net-(U1-VCAP_1)
- U1 pad 47: unconnected-(U1-VCAP_2-Pad47) -> Net-(U1-VCAP_2)
Routing:
- net VBAT+: track 45.8 -> 8.44 mm, vias 2 -> 1
- net SWDIO: track 1.34 -> 32.4 mm
- net SWCLK: track 1.57 -> 31.0 mm
- net RX4: track 5.03 -> 32.2 mm, vias 2 -> 4
- net I2C1_SCL: track 4.38 -> 27.8 mm, vias 3 -> 2
- net TX4: track 5.43 -> 28.6 mm, vias 2 -> 4
- net CURR_EXT: track 0.00 -> 23.0 mm, vias 1 -> 2
- net I2C1_SDA: track 2.78 -> 20.3 mm, vias 1 -> 3
- net M7: track 39.7 -> 30.9 mm
- net GND: track 9.34 -> 18.0 mm, vias 14 -> 22
- net SERVO_2: track 19.5 -> 11.1 mm, vias 2 -> 4
- net M6: track 36.8 -> 30.9 mm
- net M3: track 45.6 -> 41.3 mm
- net M1: track 46.3 -> 42.7 mm
- net M2: track 46.9 -> 44.0 mm
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
Commit message: Got `hwdet.dat` file mostly complete. Can compile everything now
Parts:
- added kibuzzard-66E556E1: G***, kibuzzard-66E556E1, F.Cu at (154.4, 129.4)
- added kibuzzard-66E556E7: G***, kibuzzard-66E556E7, F.Cu at (153.6, 133.1)
- added kibuzzard-66E5570F: G***, kibuzzard-66E5570F, F.Cu at (153.5, 112.2)
- added kibuzzard-66E55715: G***, kibuzzard-66E55715, F.Cu at (154.4, 116.0)
- U1: value STM32F405RGTx -> STM32F405RGT6
Connections:
- J17 pad 1: SERVO_1 -> SERVO_2
- J17 pad 2: RGB_LED -> SERVO_1
- J18 pad 1: SERVO_3 -> RGB_LED
- J18 pad 2: SERVO_2 -> SERVO_3
- U1 pad 27: VSUB_SENSE -> unconnected-(U1-PB1-Pad27)
- U1 pad 35: RGB_LED -> SERVO_1
- U1 pad 36: unconnected-(U1-PB15-Pad36) -> SERVO_2
- U1 pad 41: SERVO_1 -> M6
- U1 pad 42: M6 -> VSUB_SENSE
- U1 pad 50: SERVO_2 -> SERVO_3
- U1 pad 55: SERVO_3 -> RGB_LED
Routing:
- net RGB_LED: track 19.2 -> 7.98 mm
- net VSUB_SENSE: track 17.1 -> 8.38 mm
- net SERVO_2: track 11.1 -> 18.0 mm, vias 4 -> 2
- net SERVO_1: track 16.1 -> 19.2 mm
- net SERVO_3: track 7.98 -> 11.1 mm, vias 2 -> 4

Commit message: Almost done with pcb! Need final checks and some silkscreen design stuff
Parts:
- moved C25 0.65 mm to (170.2, 130.2)
- moved C4 0.30 mm to (167.1, 113.5), turned to 90 degrees
- moved J5 0.10 mm to (152.4, 113.3)
- moved J3 0.05 mm to (183.5, 113.3)
- moved J7 0.05 mm to (183.2, 115.3)
Connections:
- C1 pad 1: +3V3 -> +3.3V
- C10 pad 1: +3V3 -> +3.3V
- C11 pad 1: +3V3 -> +3.3V
- C12 pad 1: +3V3 -> +3.3V
- C13 pad 1: +3V3 -> +3.3V
- C14 pad 1: +3V3 -> +3.3V
- C15 pad 1: +3V3 -> +3.3V
- C16 pad 1: +3V3 -> +3.3V
- C5 pad 1: +3V3 -> +3.3V
- C6 pad 1: +3V3 -> +3.3V
- C9 pad 1: +3V3 -> +3.3V
- J16 pad 3: +3V3 -> +3.3V
- L1 pad 2: +3V3 -> +3.3V
- R1 pad 1: +3V3 -> +3.3V
- SW1 pad 2: +3V3 -> +3.3V
- U1 pad 1: +3V3 -> +3.3V
- U1 pad 13: +3V3 -> +3.3V
- U1 pad 19: +3V3 -> +3.3V
- U1 pad 32: +3V3 -> +3.3V
- U1 pad 48: +3V3 -> +3.3V
- U1 pad 64: +3V3 -> +3.3V
- U13 pad 8: +3V3 -> +3.3V
- U14 pad 5: +3V3 -> +3.3V
- U2 pad 1: +3V3 -> +3.3V
- U2 pad 10: +3V3 -> +3.3V
- U2 pad 6: +3V3 -> +3.3V
- U4 pad 6: +3V3 -> +3.3V
Routing:
- net +3.3V: track 0.00 -> 109.0 mm, vias 0 -> 13
- net +3V3: track 96.9 -> 0.00 mm, vias 10 -> 0
- net GND: track 18.0 -> 57.1 mm, vias 22 -> 42
- net CURR_EXT: track 23.0 -> 20.4 mm
- net VSYS: track 12.8 -> 10.3 mm, vias 1 -> 2
- net USB+: track 14.3 -> 12.0 mm
- net TX6: track 18.0 -> 16.2 mm
- net LED_GREEN: track 13.5 -> 15.1 mm
- net CURR_SENSE: track 17.2 -> 15.8 mm, vias 3 -> 2
- net VBUS: track 17.5 -> 16.1 mm
- net USB-: track 12.4 -> 11.4 mm
- net BOOT0: track 20.2 -> 19.3 mm
- net SWDIO: track 32.4 -> 31.6 mm
- net RGB_LED: track 7.98 -> 8.68 mm
- net RX2: track 10.6 -> 11.3 mm
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Other:
- board text added: "rev. A"
