File: kicad/f8-fc_rev-a/motors.kicad_sch (KiCad schematic)
At the start: 48 parts, among them J2 M1, J3 M2, J4 M3, J5 M4, J6 M5, J7 M6, J8 M7, J9 M8, Q2 2300A, Q3 2300A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

Commit message: Clenaup: Almost ready for order
Need to get the 30.5x30.5 holes into the outline as well, otherwise all looks good
Parts:
- D10, D11, D12, D5, D6, D7, D8, D9: LCSC Part (none) -> C455040; LSCS Part C455040 -> (none)
Changed lines of the file:
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@@
 			)
 		)
-		(property "LSCS Part" "C455040"
+		(property "LCSC Part" "C455040"
 			(at 93.98 124.46 0)
 			(effects
@@
 			)
 		)
-		(property "LSCS Part" "C455040"
+		(property "LCSC Part" "C455040"
 			(at 162.56 124.46 0)
 			(effects
@@
 			)
 		)
-		(property "LSCS Part" "C455040"
+		(property "LCSC Part" "C455040"
 			(at 199.39 124.46 0)
 			(effects
@@
 			)
 		)
-		(property "LSCS Part" "C455040"
+		(property "LCSC Part" "C455040"
 			(at 128.27 67.31 0)
 			(effects
@@
 			)
 		)
-		(property "LSCS Part" "C455040"
+		(property "LCSC Part" "C455040"
 			(at 163.83 67.31 0)
 			(effects
@@
 			)
 		)
-		(property "LSCS Part" "C455040"
+		(property "LCSC Part" "C455040"
 			(at 93.98 67.31 0)
 			(effects
@@
 			)
 		)
-		(property "LSCS Part" "C455040"
+		(property "LCSC Part" "C455040"
 			(at 199.39 67.31 0)
 			(effects
@@
 			)
 		)
-		(property "LSCS Part" "C455040"
+		(property "LCSC Part" "C455040"
 			(at 128.27 124.46 0)
 			(effects
