File: kicad/f8-fc_rev-a/f8-fc_rev-a.kicad_sch (KiCad schematic)
At the start: 57 parts, among them J1 Battery, J10 USART1, J11 USART2, J12 FC-ESC con, J13 Motors2, J14 UART4, J15 USART6, J16 I2C, J17 I2C, J18 I2C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

Commit message: Renamed project to "f8 fc"
Other:
- company: (none) -> Victor Krook
- title: (none) -> f8 fc
Changed lines of the file:
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@@
 	(generator_version "8.0")
 	(paper "A3")
+	(title_block
+		(title "f8 fc")
+		(date "2024-09-15")
+		(rev "A")
+		(company "Victor Krook")
+	)
 	(junction
 		(at 96.52 43.18)
@@
 		)
 		(instances
-			(project "fc-brushed-aio-rev-a"
+			(project "f8-fc_rev-a"
 				(path "/8f01143f-5b73-42b2-b3d1-25cdb08a54e7"
 					(page "2")

Commit message: Clenaup: Almost ready for order
Need to get the 30.5x30.5 holes into the outline as well, otherwise all looks good
Parts:
- D4: LCSC Part (none) -> C455040; LSCS Part C455040 -> (none)
Changed lines of the file:
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@@
 			)
 		)
-		(property "LSCS Part" "C455040"
+		(property "LCSC Part" "C455040"
 			(at 95.25 224.79 0)
 			(effects

Commit message: rev. A is ready to order!
Other:
- note removed: "When no battery is connected, pmos is "open", allows current through from USB. When battery is attached, it closes the pmos, which stop any current from USB to go through"
- moved on the sheet: C1, C10, C2, D1, D2, D3, D4, L1, Q1, R1, R10, R11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

Commit message: Updated cap to 0603 (C2) and driver caps from 10uf to 1uf. This is because these needs to tolerate higher voltages than 10V and that isn't available at 0402 10uF..
Parts:
- C2: footprint custom:C_0402_1005Metric_NoSilk -> custom:C_0603_1608Metric_NoSilk
Changed lines of the file:
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@@
 			)
 		)
-		(property "Footprint" "custom:C_0402_1005Metric_NoSilk"
+		(property "Footprint" "custom:C_0603_1608Metric_NoSilk"
 			(at 109.22 237.49 0)
 			(effects
