File: kicad/f8-fc-h7_rev-a/power.kicad_sch (KiCad schematic)
At the start: 43 parts, among them Q1 PMOS, Q2 WST4041, Q4 WST4041, U4 LMR33630AQRNXRQ1, U6 LMR33630AQRNXRQ1, U8 LMR33630AQRNXRQ1

Commit message: Initial ethernet PHY support
Realized however that the IC chosen (DP83848TSQ/NOPB) which
pixhawk uses in their example in Bus standard 6, isn't supported by Ardupilot.
So should probably change IC
Parts:
- removed Q2: WST4041, Package_TO_SOT_SMD:SOT-23, symbol Device:Q_PMOS_GSD
Changed lines of the file:
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@@
-	)
-	(symbol
-		(lib_id "Device:Q_PMOS_GSD")
-		(at 30.48 88.9 0)
-		(unit 1)
-		(exclude_from_sim no)
-		(in_bom yes)
-		(on_board yes)
-		(dnp no)
-		(property "Reference" "Q2"
-			(at 35.56 87.376 0)
-			(effects
-				(font
-					(size 1.27 1.27)
-				)
-				(justify left)
-			)
-		)
-		(property "Value" "WST4041"
-			(at 35.56 89.535 0)
-			(effects
-				(font
-					(size 1.27 1.27)
-				)
-				(justify left)
-			)
-		)
-		(property "Footprint" "Package_TO_SOT_SMD:SOT-23"
-			(at 35.56 86.36 0)
-			(effects
-				(font
-					(size 1.27 1.27)
-				)
-				(hide yes)
-			)
-		)
-		(property "Datasheet" "https://www.lcsc.com/datasheet/lcsc_datasheet_2311241453_Shikues-SK2301AAT_C5334586.pdf"
-			(at 30.48 88.9 0)
-			(effects
-				(font
-					(size 1.27 1.27)
-				)
-				(hide yes)
-			)
-		)
-		(property "Description" ""
-			(at 30.48 88.9 0)
-			(effects
-				(font
-					(size 1.27 1.27)
-				)
-				(hide yes)
-			)
-		)
-		(property "LCSC Part" "C148357"
-			(at 30.48 88.9 0)
-			(effects
-				(font
-					(size 1.27 1.27)
-				)
-				(hide yes)
-			)
-		)
-		(property "LSCS Part" ""
-			(at 30.48 88.9 0)
-			(effects
-				(font
-					(size 1.27 1.27)
-				)
-				(hide yes)
-			)
-		)
-		(pin "1"
-		)
-		(pin "2"
-		)
-		(pin "3"
-		)
-		(instances
-			(project "f8-fc-h7_rev"
-				(path "/8f01143f-5b73-42b2-b3d1-25cdb08a54e7/bdea3925-6af7-4d78-8700-3ad7e124738f"
-					(reference "Q2")
-					(unit 1)
-				)
-			)
-		)
 	)
 	(symbol
